Commit message: Gazebo integration: added launch and controller configs

File: src/industrial_robot_arm/urdf/Robotic.xacro (robot description, xacro)
@@ -2,5 +2,5 @@
 <robot name="Robotic" xmlns:xacro="http://www.ros.org/wiki/xacro">
 <xacro:include filename="$(find industrial_robot_arm)/urdf/materials.xacro" />
-<xacro:include filename="$(find industrial_robot_arm)/urdf/Robotic.trans" />
+<!-- <xacro:include filename="$(find industrial_robot_arm)/urdf/Robotic.trans" /> -->
 <xacro:include filename="$(find industrial_robot_arm)/urdf/Robotic.gazebo" />
 <link name="base_link">

File: src/industrial_robot_arm_moveit/config/Robotic.ros2_control.xacro (robot description, xacro)
@@ -2,9 +2,14 @@
 <robot xmlns:xacro="http://www.ros.org/wiki/xacro">
     <xacro:macro name="Robotic_ros2_control" params="name initial_positions_file">
-        <xacro:property name="initial_positions" value="${load_yaml(initial_positions_file)['initial_positions']}"/>
+        <xacro:property name="initial_positions" value="${xacro.load_yaml(initial_positions_file)['initial_positions']}"/>
+        <xacro:arg name="use_gazebo" default="true"/>
         <ros2_control name="${name}" type="system">
             <hardware>
-                <!-- By default, set up controllers for simulation. This won't work on real hardware -->
-                <plugin>mock_components/GenericSystem</plugin>
+                  <xacro:if value="$(arg use_gazebo)">
+                    <plugin>gazebo_ros2_control/GazeboSystem</plugin>
+                  </xacro:if>
+                  <xacro:unless value="$(arg use_gazebo)">
+                    <plugin>mock_components/GenericSystem</plugin>
+                  </xacro:unless>
             </hardware>
             <joint name="revolute_7">

Commit message: Add MoveIt2 Cartesian demo package and update workspace

File: src/industrial_robot_arm/urdf/Robotic.xacro (robot description, xacro)
@@ -184,4 +184,9 @@
   </collision>
 </link>
+<link name="world"/>
+<joint name="world_to_base" type="fixed">
+  <parent link="world"/>
+  <child link="base_link"/>
+</joint>
 <joint name="revolute_1" type="continuous">
   <origin xyz="0.0 0.0 0.104" rpy="0 0 0"/>
